File: kicad/turn-signal-flasher-6V.kicad_pcb (KiCad board)
At the start: 2 copper layers, 21 parts, among them J1 Conn_Blade, J2 Conn_Blade, J3 Conn_Blade, Q1 BC327, Q2 IRF4905, U1 ATtiny45-20P, U2 LM337_TO220

Commit message: finalize PCB and code
Parts:
- C1, R2: moved to B.Cu
- C3: footprint Capacitor_THT:C_Disc_D3.4mm_W2.1mm_P2.50mm -> Capacitor_SMD:C_1206_3216Metric_Pad1.33x1.80mm_HandSolder; moved to B.Cu
- Q2: value IRF4905 -> YJD70P03A; footprint Package_TO_SOT_THT:TO-220-3_Horizontal_TabDown -> Package_TO_SOT_SMD:TO-252-2
- R1: value R -> 200; moved to B.Cu
- R10, R3: value R -> 1,5k; moved to B.Cu
- R11: value R -> 0,05/5W; footprint Resistor_SMD:R_1206_3216Metric_Pad1.30x1.75mm_HandSolder -> Resistor_THT:R_Axial_DIN0617_L17.0mm_D6.0mm_P20.32mm_Horizontal
- R4, R9: value R -> 3,6k; moved to B.Cu
- R5: value R -> 1k; moved to B.Cu
- R6: value R -> 330; moved to B.Cu
- R7: value R -> 150
- R8: value R -> 1,5k
- U2: value LM337_TO220 -> LM337_TO92; footprint Package_TO_SOT_THT:TO-220-3_Vertical -> Package_TO_SOT_THT:TO-92
- moved J3 72.2 mm to (130.6, 145.0)
- moved J2 62.2 mm to (130.6, 125.0)
- moved Q1 61.6 mm to (131.5, 116.7), turned to -90 degrees
- moved C1 59.0 mm to (117.5, 113.4), turned to -90 degrees
- moved Q2 58.9 mm to (120.5, 130.9), turned to -90 degrees
- moved J1 52.5 mm to (130.5, 105.0)
- moved C3 47.8 mm to (126.1, 109.0)
- moved R11 47.6 mm to (106.5, 125.8), turned to 90 degrees
- moved R7 47.4 mm to (122.5, 121.5), turned to -90 degrees
- moved R9 45.5 mm to (109.0, 118.5)
- moved R1 42.2 mm to (135.5, 118.5), turned to 90 degrees
- moved R10 41.9 mm to (114.5, 121.5), turned to -90 degrees
- moved R3 38.7 mm to (109.0, 114.5)
- moved R5 34.3 mm to (118.5, 121.5), turned to -90 degrees
- moved R2 33.9 mm to (135.5, 113.5), turned to 90 degrees
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Connections:
- Q2 pad 3: VCC -> Net-(Q2-S)
- R11 pad 1: GND -> Net-(Q2-S)
- R11 pad 2: Net-(J3-Pin_1) -> VCC
- R8 pad 1: Net-(U1-PB2) -> Net-(U1-XTAL2/PB4)
- R8 pad 2: Net-(J3-Pin_1) -> VCC
- R9 pad 1: GND -> Net-(J3-Pin_1)
- R9 pad 2: Net-(U1-PB2) -> Net-(U1-XTAL2/PB4)
- U1 pad 3: unconnected-(U1-XTAL2/PB4-Pad3) -> Net-(U1-XTAL2/PB4)
- U1 pad 7: Net-(U1-PB2) -> unconnected-(U1-PB2-Pad7)
- U2 pad 2: VEE -> GND
- U2 pad 3: GND -> VEE
Routing:
- net GND: track 0.00 -> 58.1 mm, vias 0 -> 1
- net Net-(J3-Pin_1): track 0.00 -> 25.5 mm, vias 0 -> 156
- net VEE: track 0.00 -> 25.0 mm
- net Net-(Q1-B): track 0.00 -> 17.8 mm, vias 0 -> 1
- net Net-(U1-XTAL2/PB4): track 0.00 -> 16.5 mm, vias 0 -> 1
- net Net-(U2-ADJ): track 0.00 -> 14.4 mm, vias 0 -> 2
- net Net-(Q1-E): track 0.00 -> 13.5 mm, vias 0 -> 1
- net VCC: track 0.00 -> 11.9 mm, vias 0 -> 2
- net Net-(Q2-S): track 0.00 -> 11.7 mm
- net Net-(U1-XTAL1/PB3): track 0.00 -> 6.64 mm
- net Net-(U1-PB1): track 0.00 -> 6.48 mm, vias 0 -> 1
- net Net-(Q2-G): track 0.00 -> 2.95 mm
- added copper zone on B.Cu, net Net-(J3-Pin_1)
- added copper zone on F.Cu, net Net-(J3-Pin_1)
- added copper zone on B.Cu, net VCC
Other:
- board outline added: 40 x 50 mm
- board text added: "6V"
- board text added: "GND"

Commit message: fix: overshoot of MOSFET
Parts:
- R7: value 150 -> 2,2k
Changed lines of the file:
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@@
 		(allow_soldermask_bridges_in_footprints no)
 		(tenting front back)
+		(aux_axis_origin 100 150)
+		(grid_origin 100 150)
 		(pcbplotparams
 			(layerselection 0x00000000_00000000_55555555_575555ff)
@@
 			)
 		)
-		(property "Datasheet" ""
+		(property "Datasheet" "~"
 			(at 0 0 0)
 			(layer "F.Fab")
@@
 			)
 		)
-		(property "Datasheet" ""
+		(property "Datasheet" "~"
 			(at 0 0 0)
 			(layer "F.Fab")
@@
 			)
 		)
-		(property "Datasheet" ""
+		(property "Datasheet" "~"
 			(at 0 0 90)
 			(layer "F.Fab")
@@
 			)
 		)
-		(property "Datasheet" ""
+		(property "Datasheet" "~"
 			(at 0 0 0)
 			(layer "F.Fab")
@@
 			)
 		)
-		(property "Value" "150"
+		(property "Value" "2,2k"
 			(at 0 1.83 90)
 			(layer "F.Fab")
@@
 			)
 		)
-		(property "Datasheet" ""
+		(property "Datasheet" "~"
 			(at 0 0 90)
 			(layer "F.Fab")
@@
 			)
 		)
-		(property "Datasheet" ""
+		(property "Datasheet" "~"
 			(at 0 0 90)
 			(layer "F.Fab")
@@
 			)
 		)
-		(property "Datasheet" ""
+		(property "Datasheet" "~"
 			(at 0 0 0)
 			(layer "F.Fab")
@@
 			)
 		)
-		(property "Datasheet" ""
+		(property "Datasheet" "~"
 			(at 0 0 90)
 			(layer "B.Fab")
@@
 			)
 		)
-		(property "Datasheet" ""
+		(property "Datasheet" "~"
 			(at 0 0 0)
 			(layer "B.Fab")
@@
 			)
 		)
-		(property "Datasheet" ""
+		(property "Datasheet" "~"
 			(at 0 0 0)
 			(layer "B.Fab")
@@
 			)
 		)
-		(property "Datasheet" ""
+		(property "Datasheet" "~"
 			(at 0 0 90)
 			(layer "B.Fab")
@@
 			)
 		)
-		(property "Datasheet" ""
+		(property "Datasheet" "~"
 			(at 0 0 90)
 			(layer "B.Fab")
@@
 			)
 		)
-		(property "Datasheet" ""
+		(property "Datasheet" "~"
 			(at 0 0 0)
 			(layer "B.Fab")
@@
 			)
 		)
-		(property "Datasheet" ""
+		(property "Datasheet" "~"
 			(at 0 0 90)
 			(layer "B.Fab")
@@
 			)
 		)
-		(property "Datasheet" ""
+		(property "Datasheet" "~"
 			(at 0 0 90)
 			(layer "B.Fab")
@@
 			)
 		)
-		(property "Datasheet" ""
+		(property "Datasheet" "~"
 			(at 0 0 0)
 			(layer "B.Fab")
@@
 			)
 		)
-		(property "Datasheet" ""
+		(property "Datasheet" "~"
 			(at 0 0 90)
 			(layer "B.Fab")
